File: Hardware/1x1/MM-Qwiic-Carrier-1x1.sch (EAGLE design)
At the start: 49 parts, among them J15 MICROMOD-2222-C, J2 QWIIC_RIGHT_ANGLE, U1 MCP73831, U5 AP7361C-33FGEUDFN-8

Commit message: Remove production files. Design review changes
Parts:
- removed H6, H7, H8, H9: STAND-OFF-REFLOW2.5MM_TALL, SparkFun-Hardware:STAND-OFF-REFLOW2.5MM_TALL
- removed JP1: JUMPER-SMT_2_NC_TRACE_SILK, SparkFun-Jumpers:JUMPER-SMT_2_NC_TRACE_SILK
- added D5: 3A/10V/280mV, SparkFun-DiscreteSemi:DIODE-SCHOTTKY-BAT60A
- added J4: (no value), SparkFun-Connectors:CONN_021X02_NO_SILK
- added J5: Vertical Qwiic Connector, SparkFun-Connectors:QWIIC_CONNECTOR
- added J6: (no value), SparkFun-Connectors:CONN_08NO_SILK_FEMALE_PTH
- added TP1, TP2: TEST-POINT3X5, SparkFun-Connectors:TEST-POINT3X5
- added U$5: QWIIC_BOARD_OUTLINESTANDOFF, SparkFun-Boards:QWIIC_BOARD_OUTLINESTANDOFF
Connections:
- removed net 5V: C4.1, D3.C, D4.A, JP1.2, U1.VIN
- removed net I2C_SCL: J15.I2C_SCL, J2.4
- removed net I2C_SDA: J15.I2C_SDA, J2.3
- removed net N$5: C3.1, D3.A, J3.+, U1.VBAT
- new net D0: J15.D0, J6.3
- new net D1: J15.D1/CAM_TRIG, J6.4
- new net I2C_!INT!: J15.I2C_!INT!, J6.2
- new net SCL: J15.I2C_SCL, J2.4, J5.4, TP2.1
- new net SDA: J15.I2C_SDA, J2.3, J5.3, TP1.1
- new net SPI_!CS!: J15.SPI_!CS!, J6.8
- new net SPI_CIPO: J15.SPI_SDI, J6.5
- new net SPI_COPI: J15.SPI_SDO, J6.6
- new net SPI_SCK: J15.SPI_SCK, J6.7
- new net V_BATT: C3.1, D3.A, J3.+, J4.1, U1.VBAT
- net 3.3V: now also J5.2
- net GND: now also J4.2, J5.1, J6.1; no longer H6.1, H7.1, H8.1, H9.1
- net N$3: now also D4.C; no longer U1.STAT
- net N$8: now also U1.STAT; no longer D4.C
- net VIN: now also D3.C, D5.C; no longer JP1.1
- net V_USB: now also C4.1, D4.A, D5.A, U1.VIN
Other:
- note added: "Cut this jumper and use the PTH holes to measure current draw"
- note added: "Cut this jumper to remove power LED."
- note added: "Header"
- note added: "Power Source Select"
- note added: "Qwiic Stand offs"
- note added: "Qwiic bus conservative max current: 226mA"
- note added: "Test Points"
- note removed: "Cut these jumpers to remove power LEDs."
- note removed: "Stand offs"
- moved on the sheet: C3, C4, D3, D4, J2, J3, R1, R4, R5, S1, S2, U1

Commit message: Fix silk screen
Changed lines of the file:
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@@
 <?xml version="1.0" encoding="utf-8"?>
 <!DOCTYPE eagle SYSTEM "eagle.dtd">
-<eagle version="9.5.2">
+<eagle version="9.6.2">
 <drawing>
 <settings>
@@
 <instance part="TP1" gate="G$1" x="378.46" y="109.22" smashed="yes">
 <attribute name="NAME" x="375.92" y="111.76" size="1.778" layer="95" font="vector"/>
-<attribute name="VALUE" x="375.92" y="106.68" size="1.778" layer="96" font="vector"/>
 </instance>
 <instance part="TP2" gate="G$1" x="378.46" y="99.06" smashed="yes">
 <attribute name="NAME" x="375.92" y="101.6" size="1.778" layer="95" font="vector"/>
-<attribute name="VALUE" x="375.92" y="96.52" size="1.778" layer="96" font="vector"/>
 </instance>
 <instance part="J4" gate="G$1" x="307.34" y="139.7" smashed="yes" rot="R180">
@@
 <attribute name="VALUE" x="208.28" y="9.906" size="1.778" layer="96" align="top-center"/>
 </instance>
-<instance part="U$5" gate="G$1" x="416.56" y="78.74" smashed="yes"/>
+<instance part="U$5" gate="G$1" x="289.56" y="60.96" smashed="yes"/>
 </instances>
 <busses>

Commit message: Review before ordering
Connections:
- new net V_USB_2: BYP.1, D5.C, F2.1
- net VIN: no longer D5.C
- net V_USB: no longer BYP.1, F2.1
Changed lines of the file:
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@@
 <part name="BYP" library="SparkFun-Jumpers" deviceset="JUMPER-SMT_2_NO" device="_SILK" package3d_urn="urn:adsk.eagle:package:39279/1" value="JUMPER-SMT_2_NO_SILK"/>
 <part name="F2" library="SparkFun-Fuses" deviceset="PPTC" device="_6V2A" value="6V/2A"/>
-<part name="SUPPLY16" library="SparkFun-PowerSymbols" deviceset="V_USB" device=""/>
 <part name="U1" library="SparkFun-IC-Power" deviceset="MCP73831" device=""/>
 <part name="R1" library="SparkFun-Resistors" deviceset="2.2KOHM" device="-0603-1/10W-1%" value="2.2k"/>
@@
 <part name="GND26" library="SparkFun-PowerSymbols" deviceset="GND" device=""/>
 <part name="U$5" library="SparkFun-Boards" deviceset="QWIIC_BOARD_OUTLINE" device="STANDOFF"/>
+<part name="SUPPLY15" library="SparkFun-PowerSymbols" deviceset="V_USB_2" device=""/>
+<part name="SUPPLY16" library="SparkFun-PowerSymbols" deviceset="V_USB_2" device=""/>
 </parts>
 <sheets>
@@
 <attribute name="VALUE" x="241.808" y="231.394" size="1.778" layer="96" font="vector" align="top-center"/>
 </instance>
-<instance part="SUPPLY16" gate="G$1" x="233.68" y="246.38" smashed="yes">
-<attribute name="VALUE" x="233.68" y="249.174" size="1.778" layer="96" align="bottom-center"/>
-</instance>
 <instance part="U1" gate="G$1" x="256.54" y="149.86" smashed="yes">
 <attribute name="NAME" x="248.92" y="155.448" size="1.778" layer="95"/>
@@
 </instance>
 <instance part="U$5" gate="G$1" x="289.56" y="60.96" smashed="yes"/>
+<instance part="SUPPLY15" gate="G$1" x="396.24" y="147.32" smashed="yes">
+<attribute name="VALUE" x="396.24" y="150.114" size="1.778" layer="96" align="bottom-center"/>
+</instance>
+<instance part="SUPPLY16" gate="G$1" x="233.68" y="246.38" smashed="yes">
+<attribute name="VALUE" x="233.68" y="249.174" size="1.778" layer="96" align="bottom-center"/>
+</instance>
 </instances>
 <busses>
@@
 <wire x1="40.64" y1="66.04" x2="40.64" y2="68.58" width="0.1524" layer="91"/>
 <pinref part="SUPPLY5" gate="G$1" pin="V_USB"/>
-</segment>
-<segment>
-<wire x1="233.68" y1="233.68" x2="236.22" y2="233.68" width="0.1524" layer="91"/>
-<pinref part="BYP" gate="G$1" pin="1"/>
-<wire x1="236.22" y1="243.84" x2="233.68" y2="243.84" width="0.1524" layer="91"/>
-<wire x1="233.68" y1="243.84" x2="233.68" y2="233.68" width="0.1524" layer="91"/>
-<pinref part="F2" gate="F1" pin="1"/>
-<pinref part="SUPPLY16" gate="G$1" pin="V_USB"/>
-<wire x1="233.68" y1="246.38" x2="233.68" y2="243.84" width="0.1524" layer="91"/>
-<junction x="233.68" y="243.84"/>
 </segment>
 <segment>
@@
 <pinref part="D3" gate="G$1" pin="C"/>
 <wire x1="386.08" y1="157.48" x2="393.7" y2="157.48" width="0.1524" layer="91"/>
-<wire x1="393.7" y1="157.48" x2="393.7" y2="144.78" width="0.1524" layer="91"/>
-<pinref part="D5" gate="G$1" pin="C"/>
-<wire x1="393.7" y1="144.78" x2="386.08" y2="144.78" width="0.1524" layer="91"/>
 <wire x1="393.7" y1="157.48" x2="393.7" y2="160.02" width="0.1524" layer="91"/>
-<junction x="393.7" y="157.48"/>
 <pinref part="SUPPLY10" gate="G$1" pin="VIN"/>
 </segment>
@@
 </segment>
 </net>
+<net name="V_USB_2" class="0">
+<segment>
+<wire x1="233.68" y1="233.68" x2="236.22" y2="233.68" width="0.1524" layer="91"/>
+<pinref part="BYP" gate="G$1" pin="1"/>
+<wire x1="236.22" y1="243.84" x2="233.68" y2="243.84" width="0.1524" layer="91"/>
+<wire x1="233.68" y1="243.84" x2="233.68" y2="233.68" width="0.1524" layer="91"/>
+<pinref part="F2" gate="F1" pin="1"/>
+<pinref part="SUPPLY16" gate="G$1" pin="V_USB_2"/>
+<wire x1="233.68" y1="243.84" x2="233.68" y2="246.38" width="0.1524" layer="91"/>
+<junction x="233.68" y="243.84"/>
+</segment>
+<segment>
+<pinref part="D5" gate="G$1" pin="C"/>
+<wire x1="396.24" y1="144.78" x2="386.08" y2="144.78" width="0.1524" layer="91"/>
+<pinref part="SUPPLY15" gate="G$1" pin="V_USB_2"/>
+<wire x1="396.24" y1="144.78" x2="396.24" y2="147.32" width="0.1524" layer="91"/>
+</segment>
+</net>
