File: Hardware/1x1/MM-Qwiic-Carrier-1x1.brd (EAGLE design)
At the start: 80 x 35.6 mm, 87 parts, among them J15 MICROMOD-2222-C, J2 QWIIC_RIGHT_ANGLE, J5 Vertical Qwiic Connector, U1 MCP73831, U5 AP7361C-33FGEUDFN-8

Commit message: Silk screen changes
Parts:
- moved BYP 2.54 mm to (6.48, 21.6)
- moved U$7 2.43 mm to (11.7, 21.5)
- moved U$17 0.13 mm to (30.5, 30.5)
- moved U$18 0.13 mm to (30.5, 30.5), flipped to the bottom
- moved U$20 0.13 mm to (33.0, 30.7)
- moved U$21 0.13 mm to (33.0, 30.7)
Routing:
- net V_USB_2: track 9.63 -> 8.01 mm
- net VIN: track 32.0 -> 30.6 mm
Changed lines of the file:
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@@
 <?xml version="1.0" encoding="utf-8"?>
 <!DOCTYPE eagle SYSTEM "eagle.dtd">
-<eagle version="9.5.2">
+<eagle version="9.6.2">
 <drawing>
 <settings>
-<setting alwaysvectorfont="no"/>
+<setting alwaysvectorfont="yes"/>
 <setting verticaltext="up"/>
 </settings>
@@
 <attribute name="VALUE" x="16.51" y="15.367" size="0.6096" layer="28" font="vector" ratio="20" rot="MR0" align="top-center"/>
 </element>
-<element name="BYP" library="SparkFun-Jumpers" package="SMT-JUMPER_2_NO_SILK" package3d_urn="urn:adsk.eagle:package:39279/1" value="JUMPER-SMT_2_NO_SILK" x="6.35" y="19.05" smashed="yes" rot="MR180">
-<attribute name="NAME" x="6.35" y="17.907" size="0.6096" layer="26" font="vector" ratio="20" rot="MR180" align="bottom-center"/>
-<attribute name="VALUE" x="6.35" y="20.193" size="0.6096" layer="28" font="vector" ratio="20" rot="MR180" align="top-center"/>
+<element name="BYP" library="SparkFun-Jumpers" package="SMT-JUMPER_2_NO_SILK" package3d_urn="urn:adsk.eagle:package:39279/1" value="JUMPER-SMT_2_NO_SILK" x="6.477" y="21.59" smashed="yes" rot="MR180">
+<attribute name="NAME" x="6.477" y="20.447" size="0.6096" layer="26" font="vector" ratio="20" rot="MR180" align="bottom-center"/>
+<attribute name="VALUE" x="6.477" y="22.733" size="0.6096" layer="28" font="vector" ratio="20" rot="MR180" align="top-center"/>
 </element>
 <element name="F2" library="SparkFun-Fuses" package="1210" value="6V/2A" x="6.35" y="19.05" smashed="yes">
@@
 <element name="U$4" library="output" package="CHG0" value="" x="5.715" y="31.75" smashed="yes"/>
 <element name="U$6" library="output" package="#3#3V#0" value="" x="20.955" y="33.528" smashed="yes" rot="MR0"/>
-<element name="U$7" library="output" package="#BYP#0" value="" x="11.43" y="19.05" smashed="yes" rot="MR0"/>
+<element name="U$7" library="output" package="#BYP#0" value="" x="11.684" y="21.463" smashed="yes" rot="MR0"/>
 <element name="U$9" library="output" package="#MEAS#0" value="" x="16.51" y="7.874" smashed="yes" rot="MR0"/>
 <element name="TP1" library="SparkFun-Connectors" package="PAD.03X.05" value="TEST-POINT3X5" x="36.83" y="8.89" smashed="yes" rot="MR0"/>
@@
 <element name="U$36" library="buzzard_labels (1)" package="#0" value="" x="1.143" y="17.399" smashed="yes"/>
 <element name="U$37" library="buzzard_labels (1)" package="#0" value="" x="7.366" y="23.495" smashed="yes"/>
-<element name="U$17" library="output" package="#D0#0" value="" x="30.48" y="30.607" smashed="yes" rot="R90"/>
-<element name="U$18" library="output" package="#D0#0" value="" x="30.48" y="30.607" smashed="yes" rot="R90"/>
-<element name="U$20" library="output" package="#D1#0" value="" x="33.02" y="30.861" smashed="yes" rot="R90"/>
-<element name="U$21" library="output" package="#D1#0" value="" x="33.02" y="30.861" smashed="yes" rot="MR90"/>
 <element name="U$28" library="output" package="##CS##0" value="" x="43.18" y="30.48" smashed="yes" rot="R90"/>
 <element name="U$29" library="output" package="##CS##0" value="" x="43.18" y="30.48" smashed="yes" rot="MR90"/>
+<element name="U$17" library="output" package="#D0#0" value="" x="30.48" y="30.48" smashed="yes" rot="R90"/>
+<element name="U$18" library="output" package="#D0#0" value="" x="30.48" y="30.48" smashed="yes" rot="MR90"/>
+<element name="U$20" library="output" package="#D1#0" value="" x="33.02" y="30.734" smashed="yes" rot="R90"/>
+<element name="U$21" library="output" package="#D1#0" value="" x="33.02" y="30.734" smashed="yes" rot="MR90"/>
 </elements>
 <signals>
@@
 <wire x1="3.429" y1="19.05" x2="3.429" y2="16.51" width="0.4064" layer="1"/>
 <wire x1="3.429" y1="16.51" x2="3.429" y2="13.208" width="0.4064" layer="1"/>
-<wire x1="3.429" y1="19.05" x2="3.429" y2="20.574" width="0.4064" layer="16"/>
-<wire x1="3.429" y1="20.574" x2="5.207" y2="22.352" width="0.4064" layer="16"/>
-<wire x1="5.207" y1="22.352" x2="11.938" y2="22.352" width="0.4064" layer="16"/>
+<wire x1="3.429" y1="19.05" x2="3.429" y2="20.828" width="0.4064" layer="16"/>
+<wire x1="3.429" y1="20.828" x2="5.334" y2="22.733" width="0.4064" layer="16"/>
+<wire x1="8.382" y1="22.352" x2="11.938" y2="22.352" width="0.4064" layer="16"/>
+<wire x1="8.382" y1="22.352" x2="8.001" y2="22.733" width="0.4064" layer="16"/>
+<wire x1="8.001" y1="22.733" x2="5.334" y2="22.733" width="0.4064" layer="16"/>
 <via x="11.938" y="22.352" extent="1-16" drill="0.3048"/>
 <wire x1="11.938" y1="22.352" x2="13.12" y2="22.352" width="0.4064" layer="1"/>
@@
 <wire x1="7.85" y1="20.979" x2="7.747" y2="21.082" width="0.4064" layer="1"/>
 <via x="7.747" y="21.082" extent="1-16" drill="0.3048"/>
-<wire x1="7.747" y1="21.082" x2="6.7564" y2="20.0914" width="0.4064" layer="16"/>
-<wire x1="6.7564" y1="20.0914" x2="6.7564" y2="19.05" width="0.4064" layer="16"/>
+<wire x1="7.747" y1="21.082" x2="7.239" y2="21.59" width="0.4064" layer="16"/>
+<wire x1="7.239" y1="21.59" x2="6.8834" y2="21.59" width="0.4064" layer="16"/>
 <contactref element="D3" pad="C"/>
 <wire x1="10.03" y1="19.05" x2="10.238" y2="18.842" width="0.4064" layer="1"/>
@@
 <wire x1="7.5" y1="16.51" x2="6.4688125" y2="16.51" width="0.4064" layer="1"/>
 <wire x1="5.046" y1="17.306" x2="4.85" y2="17.502" width="0.4064" layer="1"/>
-<wire x1="4.85" y1="19.05" x2="4.85" y2="20.852" width="0.4064" layer="1"/>
-<wire x1="4.85" y1="20.852" x2="5.334" y2="21.336" width="0.4064" layer="1"/>
-<via x="5.334" y="21.336" extent="1-16" drill="0.381"/>
-<wire x1="5.334" y1="21.336" x2="5.9436" y2="20.7264" width="0.4064" layer="16"/>
-<wire x1="5.9436" y1="20.7264" x2="5.9436" y2="19.05" width="0.4064" layer="16"/>
+<wire x1="4.85" y1="19.05" x2="4.85" y2="20.979" width="0.4064" layer="1"/>
+<wire x1="4.85" y1="20.979" x2="5.207" y2="21.336" width="0.4064" layer="1"/>
+<via x="5.207" y="21.336" extent="1-16" drill="0.381"/>
+<wire x1="5.207" y1="21.336" x2="5.461" y2="21.59" width="0.4064" layer="16"/>
+<wire x1="6.0706" y1="21.59" x2="5.461" y2="21.59" width="0.4064" layer="16"/>
 </signal>
 </signals>

Commit message: QC Feedback
Parts:
- moved H5 0.13 mm to (44.1, 13.8)
Changed lines of the file:
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@@
 <?xml version="1.0" encoding="utf-8"?>
 <!DOCTYPE eagle SYSTEM "eagle.dtd">
-<eagle version="9.6.2">
+<eagle version="9.5.2">
 <drawing>
 <settings>
-<setting alwaysvectorfont="yes"/>
+<setting alwaysvectorfont="no"/>
 <setting verticaltext="up"/>
 </settings>
@@
 <layer number="45" name="Holes" color="7" fill="1" visible="yes" active="yes"/>
 <layer number="46" name="Milling" color="3" fill="1" visible="no" active="yes"/>
-<layer number="47" name="Measures" color="7" fill="1" visible="no" active="yes"/>
+<layer number="47" name="Measures" color="7" fill="1" visible="yes" active="yes"/>
 <layer number="48" name="Document" color="7" fill="1" visible="no" active="yes"/>
 <layer number="49" name="Reference" color="7" fill="1" visible="no" active="yes"/>
@@
 <wire x1="44.185" y1="6.731" x2="27.94" y2="6.731" width="0.2032" layer="21"/>
 <text x="36.83" y="-21.59" size="1.778" layer="51" font="vector" ratio="15">Priyanka Makin</text>
-<dimension x1="0" y1="35.56" x2="80.01" y2="35.56" x3="40.005" y3="39.37" textsize="1.778" textratio="15" layer="47" unit="inch"/>
-<dimension x1="80.01" y1="35.56" x2="80.01" y2="0" x3="83.82" y3="17.78" textsize="1.778" textratio="15" layer="47" unit="inch"/>
-<text x="43.434" y="39.878" size="1.778" layer="47" font="vector" ratio="15">in</text>
+<dimension x1="0" y1="35.56" x2="80.01" y2="35.56" x3="40.005" y3="45.72" textsize="1.778" textratio="15" layer="47" unit="inch"/>
+<dimension x1="80.01" y1="35.56" x2="80.01" y2="0" x3="91.44" y3="17.78" textsize="1.778" textratio="15" layer="47" unit="inch"/>
+<text x="43.434" y="42.418" size="1.778" layer="47" font="vector" ratio="15">in</text>
+<text x="85.344" y="23.241" size="1.778" layer="47" font="vector" ratio="15" rot="R270">in</text>
+<dimension x1="2.54" y1="33.02" x2="77.47" y2="33.02" x3="40.005" y3="41.91" textsize="1.778" textratio="15" layer="47" unit="inch"/>
+<dimension x1="77.47" y1="33.02" x2="77.47" y2="2.54" x3="87.63" y3="17.78" textsize="1.778" textratio="15" layer="47" unit="inch"/>
+<text x="43.434" y="46.228" size="1.778" layer="47" font="vector" ratio="15">in</text>
+<text x="89.154" y="23.241" size="1.778" layer="47" font="vector" ratio="15" rot="R270">in</text>
+<dimension x1="52.07" y1="27.94" x2="72.39" y2="27.94" x3="62.23" y3="38.1" textsize="1.778" textratio="15" layer="47" unit="inch"/>
+<dimension x1="72.39" y1="27.94" x2="72.39" y2="7.62" x3="83.82" y3="17.78" textsize="1.778" textratio="15" layer="47" unit="inch"/>
 <text x="81.534" y="23.241" size="1.778" layer="47" font="vector" ratio="15" rot="R270">in</text>
-<dimension x1="2.54" y1="33.02" x2="77.47" y2="33.02" x3="40.005" y3="44.45" textsize="1.778" textratio="15" layer="47" unit="inch"/>
-<dimension x1="77.47" y1="33.02" x2="77.47" y2="2.54" x3="88.9" y3="17.78" textsize="1.778" textratio="15" layer="47" unit="inch"/>
-<text x="43.434" y="44.958" size="1.778" layer="47" font="vector" ratio="15">in</text>
-<text x="86.614" y="23.241" size="1.778" layer="47" font="vector" ratio="15" rot="R270">in</text>
+<text x="65.024" y="38.608" size="1.778" layer="47" font="vector" ratio="15">in</text>
 </plain>
 <attributes>
@@
 <element name="LOGO3" library="SparkFun-Aesthetics" package="OSHW-LOGO-M" value="OSHW-LOGOM" x="31.623" y="10.922" smashed="yes" rot="MR0"/>
 <element name="U$55" library="buzzard_labels (9)" package="22229" value="" x="26.962" y="5.72" smashed="yes"/>
-<element name="H5" library="SparkFun-Hardware" package="STAND-OFF-REFLOW-M2.5" value="STAND-OFF-REFLOW2.5MM_TALL" x="44.2" y="13.76" smashed="yes">
-<attribute name="PROD_ID" value="HW-14899" x="44.2" y="13.76" size="1.778" layer="27" font="vector" ratio="15" display="off"/>
+<element name="H5" library="SparkFun-Hardware" package="STAND-OFF-REFLOW-M2.5" value="STAND-OFF-REFLOW2.5MM_TALL" x="44.073" y="13.76" smashed="yes">
+<attribute name="PROD_ID" value="HW-14899" x="44.073" y="13.76" size="1.778" layer="27" font="vector" ratio="15" display="off"/>
 </element>
 <element name="JP4" library="SparkFun-Jumpers" package="SMT-JUMPER_2_NC_TRACE_SILK" package3d_urn="urn:adsk.eagle:package:39281/1" value="3V3 LED" x="15.24" y="33.655" smashed="yes" rot="MR0">
