File: Hardware/2x1/MM-Qwiic-Carrier-2x1.brd (EAGLE design)
At the start: 108 x 35.6 mm, 88 parts, among them J15 MICROMOD-2222-C, J2 QWIIC_RIGHT_ANGLE, J5 Vertical Qwiic Connector, U1 MCP73831, U5 AP7361C-33FGEUDFN-8

Commit message: Silk screen changes
Parts:
- moved BYP 2.54 mm to (6.48, 21.6)
- moved U$7 2.43 mm to (11.7, 21.5)
- moved FD2 1.27 mm to (105.9, 34.9)
- moved FD4 1.27 mm to (105.9, 34.9)
- moved H1 1.27 mm to (104.1, 33.0)
- moved H3 1.27 mm to (104.1, 2.54)
- moved U$31 0.64 mm to (65.7, 2.54)
- moved U$34 0.13 mm to (42.8, 16.8)
- moved U$17 0.13 mm to (30.5, 30.5)
- moved U$18 0.13 mm to (30.5, 30.5), flipped to the bottom
- moved U$20 0.13 mm to (33.0, 30.7)
- moved U$21 0.13 mm to (33.0, 30.7)
Routing:
- net V_USB_2: track 9.63 -> 8.01 mm
- net VIN: track 32.0 -> 30.6 mm
Other:
- board size 108 x 35.6 mm -> 106.7 x 35.6 mm
