File: Hardware/Single/MM-Qwiic-Carrier-Single.brd (EAGLE design)
At the start: 80 x 35.6 mm, 89 parts, among them J15 MICROMOD-2222-C, J2 QWIIC_RIGHT_ANGLE, J5 Vertical Qwiic Connector, U1 MCP73831, U5 AP7361C-33FGEUDFN-8

Commit message: Move SF logo, board name silk screen on bottom
Renamed eagle files from 1x1, 2x1 to single, double
Cleaned up library files
Parts:
- moved LOGO3 30.6 mm to (62.2, 9.91)
- moved U$19 30.5 mm to (75.1, 16.0)
- moved LOGO1 30.5 mm to (62.2, 20.8)
- moved U$68 30.5 mm to (62.2, 18.2)
Changed lines of the file:
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@@
 <?xml version="1.0" encoding="utf-8"?>
 <!DOCTYPE eagle SYSTEM "eagle.dtd">
-<eagle version="9.6.2">
+<eagle version="9.5.2">
 <drawing>
 <settings>
@@
 </element>
 <element name="LOGO2" library="SparkFun-Aesthetics" package="QWIIC_5.5MM" value="QWIIC_LOGO_CONNECTOR" x="33.401" y="3.1115" smashed="yes" rot="R90"/>
-<element name="LOGO3" library="SparkFun-Aesthetics" package="OSHW-LOGO-M" value="OSHW-LOGOM" x="31.623" y="10.922" smashed="yes" rot="MR0"/>
+<element name="LOGO3" library="SparkFun-Aesthetics" package="OSHW-LOGO-M" value="OSHW-LOGOM" x="62.23" y="9.906" smashed="yes" rot="MR0"/>
 <element name="H5" library="SparkFun-Hardware" package="STAND-OFF-REFLOW-M2.5" value="STAND-OFF-REFLOW2.5MM_TALL" x="44.073" y="13.76" smashed="yes">
 <attribute name="PROD_ID" value="HW-14899" x="44.073" y="13.76" size="1.778" layer="27" font="vector" ratio="15" display="off"/>
@@
 <attribute name="VALUE" x="23.495" y="17.78" size="0.762" layer="27" rot="R270" align="center"/>
 </element>
-<element name="LOGO1" library="SparkFun-Aesthetics" package="SFE_LOGO_NAME_FLAME_.2" value="SFE_LOGO_NAME_FLAME.2_INCH" x="31.75" y="22.098" smashed="yes" rot="MR0"/>
+<element name="LOGO1" library="SparkFun-Aesthetics" package="SFE_LOGO_NAME_FLAME_.2" value="SFE_LOGO_NAME_FLAME.2_INCH" x="62.23" y="20.828" smashed="yes" rot="MR0"/>
 <element name="U$44" library="SparkFun-Aesthetics" package="SFE_LOGO_FLAME_.2" value="" x="18.034" y="30.607" smashed="yes"/>
 <element name="U$67" library="SparkFun-MicroMod" package="MICROMOD_LOGO_.5" value="" x="62.103" y="33.401" smashed="yes"/>
-<element name="U$68" library="SparkFun-MicroMod" package="MICROMOD_LOGO_.5" value="" x="31.75" y="19.431" smashed="yes" rot="MR0"/>
+<element name="U$68" library="SparkFun-MicroMod" package="MICROMOD_LOGO_.5" value="" x="62.23" y="18.161" smashed="yes" rot="MR0"/>
 <element name="J2" library="SparkFun-Connectors" package="JST04_1MM_RA" value="QWIIC_RIGHT_ANGLE" x="38.1" y="5.08" smashed="yes">
 <attribute name="NAME" x="36.703" y="2.921" size="0.6096" layer="25" font="vector" ratio="20"/>
@@
 <element name="U$16" library="output" package="##INT##0" value="" x="27.94" y="29.845" smashed="yes" rot="MR90"/>
 <element name="U$2" library="output" package="QWIIC_CARRIER_#_SINGLE0" value="" x="49.53" y="2.54" smashed="yes"/>
-<element name="U$19" library="output" package="QWIIC_CARRIER_#_SINGLE0" value="" x="44.577" y="17.272" smashed="yes" rot="MR0"/>
+<element name="U$19" library="output" package="QWIIC_CARRIER_#_SINGLE0" value="" x="75.057" y="16.002" smashed="yes" rot="MR0"/>
 </elements>
 <signals>
