File: Hardware/Double/Production/MM-Qwiic-Carrier-2x1-Panel.brd (EAGLE design)
At the start: 180.6 x 158 mm, 710 parts, among them J12 Vertical Qwiic Connector, J15 MICROMOD-2222-C, J16 MICROMOD-2222-C, J17 QWIIC_RIGHT_ANGLE, J2 QWIIC_RIGHT_ANGLE, J20 Vertical Qwiic Connector, J23 MICROMOD-2222-C, J24 QWIIC_RIGHT_ANGLE, J27 Vertical Qwiic Connector, J30 MICROMOD-2222-C, J31 QWIIC_RIGHT_ANGLE, J34 Vertical Qwiic Connector, J37 MICROMOD-2222-C, J38 QWIIC_RIGHT_ANGLE, J41 Vertical Qwiic Connector, J44 MICROMOD-2222-C, J45 QWIIC_RIGHT_ANGLE, J48 Vertical Qwiic Connector, J5 Vertical Qwiic Connector, J51 MICROMOD-2222-C, J52 QWIIC_RIGHT_ANGLE, J55 Vertical Qwiic Connector, J8 MICROMOD-2222-C, J9 QWIIC_RIGHT_ANGLE, U1 MCP73831, U10 MCP73831, U11 AP7361C-33FGEUDFN-8, U12 MCP73831, U13 AP7361C-33FGEUDFN-8, U14 MCP73831, U15 AP7361C-33FGEUDFN-8, U16 MCP73831, U2 AP7361C-33FGEUDFN-8, U3 MCP73831, U4 AP7361C-33FGEUDFN-8, U5 AP7361C-33FGEUDFN-8, U6 MCP73831, U7 AP7361C-33FGEUDFN-8, U8 MCP73831, U9 AP7361C-33FGEUDFN-8

Commit message: Renaming
1x1 --> Single
2x1 --> Double
Re-panelized
Parts:
- added U$313: (no value), output:#3#3V#0
- added U$314, U$315: (no value), output:##CS##0
- added U$316, U$317: (no value), output:##INT##0
- added U$318: QWIIC_BOARD_OUTLINESTANDOFF, SparkFun-Boards:QWIIC_BOARD_MOUNT_SMD_STANDOFFS
- added U$319, U$320: (no value), output:QWIIC_CARRIER_#_DOUBLE0
- U$10, U$13: device output:QWIIC_CARRIER_#_1X10 -> output:QWIIC_CARRIER_#_DOUBLE0
- U$118, U$2: value (none) -> QWIIC_BOARD_OUTLINESTANDOFF; device SparkFun-Aesthetics:SFE_LOGO_FLAME_.2 -> SparkFun-Boards:QWIIC_BOARD_MOUNT_SMD_STANDOFFS
- U$119, U$120, U$159, U$80: device SparkFun-MicroMod:MICROMOD_LOGO_.5 -> output:QWIIC_CARRIER_#_DOUBLE0
- U$121: device output:CHG0 -> SparkFun-Aesthetics:SFE_LOGO_FLAME_.2
- U$122, U$83: device output:#3#3V#0 -> SparkFun-MicroMod:MICROMOD_LOGO_.5
- U$123, U$162: device output:#BYP#0 -> SparkFun-MicroMod:MICROMOD_LOGO_.5
- U$124: device output:#MEAS#0 -> output:CHG0
- U$125: value QWIIC_BOARD_OUTLINESTANDOFF -> (none); device SparkFun-Boards:QWIIC_BOARD_MOUNT_SMD_STANDOFFS -> output:#3#3V#0
- U$126, U$166: device output:QWIIC_CARRIER_#_1X10 -> output:#BYP#0
- U$127, U$87: device output:QWIIC_CARRIER_#_1X10 -> output:#MEAS#0
- U$128: value (none) -> QWIIC_BOARD_OUTLINESTANDOFF; device output:3V30 -> SparkFun-Boards:QWIIC_BOARD_MOUNT_SMD_STANDOFFS
- U$129: device output:#3#3V_EN#0 -> output:3V30
- U$130, U$170: device output:#GND#0 -> output:#3#3V_EN#0
- U$132, U$171, U$172, U$211: device output:#CIPO#0 -> output:#GND#0
- U$134, U$173, U$174, U$213: device output:#COPI#0 -> output:#CIPO#0
- U$136, U$175, U$176, U$215: device output:#SCK#0 -> output:#COPI#0
- U$138, U$177: device output:#VBAT#0 -> output:#SCK#0
- U$139: device output:#GND#0 -> output:#VBAT#0
- U$140, U$180: device output:#0 -> output:#GND#0
- U$142, U$181, U$182, U$221: device buzzard_labels (1):#0 -> output:#0
- U$144, U$183, U$184, U$223: device output:#D0#0 -> buzzard_labels (1):#0
- U$146, U$185, U$186, U$225: device output:#D1#0 -> output:#D0#0
- U$148, U$187: device output:RESET0 -> output:#D1#0
- U$149: device output:BOOT0 -> output:RESET0
- U$150: device output:22220 -> output:BOOT0
- U$151, U$191: device output:#3#3V#0 -> output:22220
- U$153, U$192, U$193, U$232: device output:##CS##0 -> output:#3#3V#0
- U$155, U$194, U$195, U$234: device output:##INT##0 -> output:##CS##0
- U$157, U$196: device SparkFun-Aesthetics:SFE_LOGO_FLAME_.2 -> output:##INT##0
- U$158, U$198: value (none) -> QWIIC_BOARD_OUTLINESTANDOFF; device SparkFun-MicroMod:MICROMOD_LOGO_.5 -> SparkFun-Boards:QWIIC_BOARD_MOUNT_SMD_STANDOFFS
- U$160, U$199: device output:CHG0 -> output:QWIIC_CARRIER_#_DOUBLE0
- U$161: device output:#3#3V#0 -> SparkFun-Aesthetics:SFE_LOGO_FLAME_.2
- U$163, U$202: device output:#MEAS#0 -> SparkFun-MicroMod:MICROMOD_LOGO_.5
- U$164: value QWIIC_BOARD_OUTLINESTANDOFF -> (none); device SparkFun-Boards:QWIIC_BOARD_MOUNT_SMD_STANDOFFS -> output:CHG0
- U$165, U$205: device output:QWIIC_CARRIER_#_1X10 -> output:#3#3V#0
- U$167: device output:3V30 -> output:#MEAS#0
- U$168: value (none) -> QWIIC_BOARD_OUTLINESTANDOFF; device output:#3#3V_EN#0 -> SparkFun-Boards:QWIIC_BOARD_MOUNT_SMD_STANDOFFS
- U$169, U$209: device output:#GND#0 -> output:3V30
- U$178, U$217: device output:#GND#0 -> output:#SCK#0
- U$179, U$219: device output:#0 -> output:#VBAT#0
- U$188, U$227: device output:BOOT0 -> output:#D1#0
- U$189: device output:22220 -> output:RESET0
- U$19, U$81: device SparkFun-MicroMod:MICROMOD_LOGO_.5 -> SparkFun-Aesthetics:SFE_LOGO_FLAME_.2
- U$190, U$230: device output:#3#3V#0 -> output:BOOT0
- U$197, U$236, U$237, U$276: device SparkFun-MicroMod:MICROMOD_LOGO_.5 -> output:##INT##0
- U$200, U$239: device output:#3#3V#0 -> output:QWIIC_CARRIER_#_DOUBLE0
- U$201: device output:#BYP#0 -> SparkFun-Aesthetics:SFE_LOGO_FLAME_.2
- U$203, U$242: value QWIIC_BOARD_OUTLINESTANDOFF -> (none); device SparkFun-Boards:QWIIC_BOARD_MOUNT_SMD_STANDOFFS -> SparkFun-MicroMod:MICROMOD_LOGO_.5
- U$204, U$244: device output:QWIIC_CARRIER_#_1X10 -> output:CHG0
- U$206: device output:3V30 -> output:#BYP#0
- U$207: device output:#3#3V_EN#0 -> output:#MEAS#0
- U$208, U$248: value (none) -> QWIIC_BOARD_OUTLINESTANDOFF; device output:#GND#0 -> SparkFun-Boards:QWIIC_BOARD_MOUNT_SMD_STANDOFFS
- U$210, U$250: device output:#CIPO#0 -> output:#3#3V_EN#0
- U$212, U$251, U$252, U$291: device output:#COPI#0 -> output:#GND#0
- U$214, U$253, U$254, U$293: device output:#SCK#0 -> output:#CIPO#0
- U$216, U$255: device output:#VBAT#0 -> output:#COPI#0
- U$218, U$257, U$258, U$297: device output:#0 -> output:#SCK#0
- U$220, U$260: device buzzard_labels (1):#0 -> output:#GND#0
- U$222, U$261, U$262, U$301: device output:#D0#0 -> output:#0
- U$224, U$263, U$264, U$303: device output:#D1#0 -> buzzard_labels (1):#0
- U$226, U$265: device output:RESET0 -> output:#D0#0
- U$228, U$267: device output:22220 -> output:#D1#0
- U$229, U$269: device output:#3#3V#0 -> output:RESET0
- U$231, U$271: device output:##CS##0 -> output:22220
- U$233, U$272, U$273, U$312: device output:##INT##0 -> output:#3#3V#0
- U$235, U$274: device SparkFun-Aesthetics:SFE_LOGO_FLAME_.2 -> output:##CS##0
- U$238: value (none) -> QWIIC_BOARD_OUTLINESTANDOFF; device output:CHG0 -> SparkFun-Boards:QWIIC_BOARD_MOUNT_SMD_STANDOFFS
- U$240, U$279: device output:#BYP#0 -> output:QWIIC_CARRIER_#_DOUBLE0
- U$241: device output:#MEAS#0 -> SparkFun-Aesthetics:SFE_LOGO_FLAME_.2
- U$243, U$282, U$283: device output:QWIIC_CARRIER_#_1X10 -> SparkFun-MicroMod:MICROMOD_LOGO_.5
- U$245: device output:3V30 -> output:#3#3V#0
- U$246: device output:#3#3V_EN#0 -> output:#BYP#0
- U$247, U$287: device output:#GND#0 -> output:#MEAS#0
- U$249, U$289: device output:#CIPO#0 -> output:3V30
- U$256, U$295: device output:#GND#0 -> output:#COPI#0
- U$259, U$299: device buzzard_labels (1):#0 -> output:#VBAT#0
- U$266, U$305: device output:BOOT0 -> output:#D0#0
- U$268, U$307, U$308: device output:#3#3V#0 -> output:#D1#0
- U$270, U$310: device output:##CS##0 -> output:BOOT0
- U$275: device SparkFun-MicroMod:MICROMOD_LOGO_.5 -> output:##CS##0
- U$277: device output:CHG0 -> output:##INT##0
- U$278: value (none) -> QWIIC_BOARD_OUTLINESTANDOFF; device output:#3#3V#0 -> SparkFun-Boards:QWIIC_BOARD_MOUNT_SMD_STANDOFFS
- U$280: device output:#MEAS#0 -> output:QWIIC_CARRIER_#_DOUBLE0
- U$281: value QWIIC_BOARD_OUTLINESTANDOFF -> (none); device SparkFun-Boards:QWIIC_BOARD_MOUNT_SMD_STANDOFFS -> SparkFun-Aesthetics:SFE_LOGO_FLAME_.2
- U$284: device output:3V30 -> output:CHG0
- U$285: device output:#3#3V_EN#0 -> output:#3#3V#0
- U$286: device output:#GND#0 -> output:#BYP#0
- U$288: value (none) -> QWIIC_BOARD_OUTLINESTANDOFF; device output:#CIPO#0 -> SparkFun-Boards:QWIIC_BOARD_MOUNT_SMD_STANDOFFS
- U$290: device output:#COPI#0 -> output:#3#3V_EN#0
- U$292: device output:#SCK#0 -> output:#GND#0
- U$294: device output:#VBAT#0 -> output:#CIPO#0
- U$296: device output:#0 -> output:#COPI#0
- U$298: device buzzard_labels (1):#0 -> output:#SCK#0
- U$300: device output:#D0#0 -> output:#GND#0
- U$302: device output:#D1#0 -> output:#0
- U$304: device output:RESET0 -> buzzard_labels (1):#0
- U$306: device output:22220 -> output:#D0#0
- U$309: device output:##CS##0 -> output:RESET0
- U$311: device output:##INT##0 -> output:22220
- U$40, U$82: device output:CHG0 -> SparkFun-MicroMod:MICROMOD_LOGO_.5
- U$41: device output:#3#3V#0 -> output:CHG0
- U$42: device output:#BYP#0 -> output:#3#3V#0
- U$43: device output:#MEAS#0 -> output:#BYP#0
- U$45: value QWIIC_BOARD_OUTLINESTANDOFF -> (none); device SparkFun-Boards:QWIIC_BOARD_MOUNT_SMD_STANDOFFS -> output:#MEAS#0
- U$46, U$88: value (none) -> QWIIC_BOARD_OUTLINESTANDOFF; device output:QWIIC_CARRIER_#_1X10 -> SparkFun-Boards:QWIIC_BOARD_MOUNT_SMD_STANDOFFS
- U$47: device output:QWIIC_CARRIER_#_1X10 -> output:3V30
- U$48: device output:3V30 -> output:#3#3V_EN#0
- U$49: device output:#3#3V_EN#0 -> output:#GND#0
- U$51: device output:#GND#0 -> output:#CIPO#0
- U$53: device output:#CIPO#0 -> output:#COPI#0
- U$55: device output:#COPI#0 -> output:#SCK#0
- U$57: device output:#SCK#0 -> output:#VBAT#0
- U$58: device output:#VBAT#0 -> output:#GND#0
- U$59: device output:#GND#0 -> output:#0
- U$61: device output:#0 -> buzzard_labels (1):#0
- U$63: device buzzard_labels (1):#0 -> output:#D0#0
- U$65: device output:#D0#0 -> output:#D1#0
- U$69: device output:#D1#0 -> output:RESET0
- U$70: device output:RESET0 -> output:BOOT0
- U$71: device output:BOOT0 -> output:22220
- U$72: device output:22220 -> output:#3#3V#0
- U$74: device output:#3#3V#0 -> output:##CS##0
- U$76: device output:##CS##0 -> output:##INT##0
- U$78: value (none) -> QWIIC_BOARD_OUTLINESTANDOFF; device output:##INT##0 -> SparkFun-Boards:QWIIC_BOARD_MOUNT_SMD_STANDOFFS
- U$79: device SparkFun-Aesthetics:SFE_LOGO_FLAME_.2 -> output:QWIIC_CARRIER_#_DOUBLE0
- U$84: device output:#BYP#0 -> output:CHG0
- U$85: device output:#MEAS#0 -> output:#3#3V#0
- U$86: value QWIIC_BOARD_OUTLINESTANDOFF -> (none); device SparkFun-Boards:QWIIC_BOARD_MOUNT_SMD_STANDOFFS -> output:#BYP#0
- moved U$238 203.0 mm to (202.4, 89.9)
- moved U$79 168.6 mm to (174.0, 2.54)
- moved U$239 167.1 mm to (174.0, 74.7), flipped to the top
- moved U$160 157.2 mm to (154.7, 53.7), flipped to the bottom
- moved U$159 151.6 mm to (174.0, 38.6), flipped to the top
- moved U$158 149.6 mm to (202.4, 53.8)
- moved U$240 148.5 mm to (154.7, 89.8)
- moved U$235 139.6 mm to (152.9, 102.6), flipped to the bottom, turned to 90 degrees
- moved U$157 125.2 mm to (137.7, 65.9), flipped to the bottom, turned to 90 degrees
- moved U$197 114.7 mm to (27.9, 102.0), flipped to the bottom, turned to 90 degrees
- moved U$237 108.9 mm to (137.7, 102.0), turned to 90 degrees
- moved U$80 106.1 mm to (154.7, 17.7), flipped to the bottom
- moved U$275 99.5 mm to (43.2, 138.7), flipped to the bottom, turned to 90 degrees
- moved U$78 94.8 mm to (202.4, 17.8), flipped to the top, turned to 0 degrees
- moved U$202 93.6 mm to (187.1, 105.5), flipped to the top
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Other:
- board size 180.6 x 158 mm -> 239 x 158 mm
