File: Hardware/Double/Production/MM-Qwiic-Carrier-Double-Panel.brd (EAGLE design)
At the start: 239 x 158 mm, 718 parts, among them J12 Vertical Qwiic Connector, J15 MICROMOD-2222-C, J16 MICROMOD-2222-C, J17 QWIIC_RIGHT_ANGLE, J2 QWIIC_RIGHT_ANGLE, J20 Vertical Qwiic Connector, J23 MICROMOD-2222-C, J24 QWIIC_RIGHT_ANGLE, J27 Vertical Qwiic Connector, J30 MICROMOD-2222-C, J31 QWIIC_RIGHT_ANGLE, J34 Vertical Qwiic Connector, J37 MICROMOD-2222-C, J38 QWIIC_RIGHT_ANGLE, J41 Vertical Qwiic Connector, J44 MICROMOD-2222-C, J45 QWIIC_RIGHT_ANGLE, J48 Vertical Qwiic Connector, J5 Vertical Qwiic Connector, J51 MICROMOD-2222-C, J52 QWIIC_RIGHT_ANGLE, J55 Vertical Qwiic Connector, J8 MICROMOD-2222-C, J9 QWIIC_RIGHT_ANGLE, U1 MCP73831, U10 MCP73831, U11 AP7361C-33FGEUDFN-8, U12 MCP73831, U13 AP7361C-33FGEUDFN-8, U14 MCP73831, U15 AP7361C-33FGEUDFN-8, U16 MCP73831, U2 AP7361C-33FGEUDFN-8, U3 MCP73831, U4 AP7361C-33FGEUDFN-8, U5 AP7361C-33FGEUDFN-8, U6 MCP73831, U7 AP7361C-33FGEUDFN-8, U8 MCP73831, U9 AP7361C-33FGEUDFN-8

Commit message: Re-panelized with corrected position silk screen
This is the last time I've got to re-panel hopefully!
Parts:
- moved U$120 61.0 mm to (105.9, 51.2)
- moved U$13 61.0 mm to (105.9, 15.1)
- moved U$200 61.0 mm to (105.9, 87.2)
- moved U$280 61.0 mm to (105.9, 123.3)
- moved LOGO1 61.0 mm to (92.7, 19.7)
- moved LOGO15 61.0 mm to (92.7, 91.8)
- moved LOGO21 61.0 mm to (92.7, 127.9)
- moved LOGO9 61.0 mm to (92.7, 55.8)
- moved U$163 61.0 mm to (92.7, 89.3)
- moved U$243 61.0 mm to (92.7, 125.3)
- moved U$68 61.0 mm to (92.7, 17.1)
- moved U$83 61.0 mm to (92.7, 53.2)
- moved LOGO12 61.0 mm to (202.4, 55.8)
- moved LOGO18 61.0 mm to (202.4, 91.8)
- moved LOGO24 61.0 mm to (202.4, 127.9)
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