File: Hardware/Single/Production/MM-Qwiic-Carrier-1x1-Panel.brd (EAGLE design)
At the start: 239 x 158 mm, 718 parts, among them J12 Vertical Qwiic Connector, J15 MICROMOD-2222-C, J16 MICROMOD-2222-C, J17 QWIIC_RIGHT_ANGLE, J2 QWIIC_RIGHT_ANGLE, J20 Vertical Qwiic Connector, J23 MICROMOD-2222-C, J24 QWIIC_RIGHT_ANGLE, J27 Vertical Qwiic Connector, J30 MICROMOD-2222-C, J31 QWIIC_RIGHT_ANGLE, J34 Vertical Qwiic Connector, J37 MICROMOD-2222-C, J38 QWIIC_RIGHT_ANGLE, J41 Vertical Qwiic Connector, J44 MICROMOD-2222-C, J45 QWIIC_RIGHT_ANGLE, J48 Vertical Qwiic Connector, J5 Vertical Qwiic Connector, J51 MICROMOD-2222-C, J52 QWIIC_RIGHT_ANGLE, J55 Vertical Qwiic Connector, J8 MICROMOD-2222-C, J9 QWIIC_RIGHT_ANGLE, U1 MCP73831, U10 MCP73831, U11 AP7361C-33FGEUDFN-8, U12 MCP73831, U13 AP7361C-33FGEUDFN-8, U14 MCP73831, U15 AP7361C-33FGEUDFN-8, U16 MCP73831, U2 AP7361C-33FGEUDFN-8, U3 MCP73831, U4 AP7361C-33FGEUDFN-8, U5 AP7361C-33FGEUDFN-8, U6 MCP73831, U7 AP7361C-33FGEUDFN-8, U8 MCP73831, U9 AP7361C-33FGEUDFN-8

Commit message: Renaming
1x1 --> Single
2x1 --> Double
Re-panelized
Parts:
- removed U$313: (no value), output:#3#3V#0
- removed U$314, U$315: (no value), output:##CS##0
- removed U$316, U$317: (no value), output:##INT##0
- removed U$318: QWIIC_BOARD_OUTLINESTANDOFF, SparkFun-Boards:QWIIC_BOARD_MOUNT_SMD_STANDOFFS
- removed U$319, U$320: (no value), output:QWIIC_CARRIER_#_2X10
- U$100, U$58: device output:#GND#0 -> output:#0
- U$101, U$102, U$141, U$60: device output:#0 -> buzzard_labels (1):#0
- U$103, U$104, U$143, U$62: device buzzard_labels (1):#0 -> output:#D0#0
- U$105, U$106, U$145, U$64: device output:#D0#0 -> output:#D1#0
- U$107, U$66: device output:#D1#0 -> output:RESET0
- U$108, U$147: device output:#D1#0 -> output:BOOT0
- U$109: device output:RESET0 -> output:22220
- U$110, U$150: device output:BOOT0 -> output:#3#3V#0
- U$111, U$71: device output:22220 -> output:#3#3V#0
- U$112, U$113, U$152, U$73: device output:#3#3V#0 -> output:##CS##0
- U$114, U$115, U$154, U$75: device output:##CS##0 -> output:##INT##0
- U$116, U$117, U$156, U$77: device output:##INT##0 -> output:QWIIC_CARRIER_#_SINGLE0
- U$118: value QWIIC_BOARD_OUTLINESTANDOFF -> (none); device SparkFun-Boards:QWIIC_BOARD_MOUNT_SMD_STANDOFFS -> SparkFun-Aesthetics:SFE_LOGO_FLAME_.2
- U$119, U$120, U$159, U$39, U$80: device output:QWIIC_CARRIER_#_2X10 -> SparkFun-MicroMod:MICROMOD_LOGO_.5
- U$121: device SparkFun-Aesthetics:SFE_LOGO_FLAME_.2 -> output:CHG0
- U$122, U$83: device SparkFun-MicroMod:MICROMOD_LOGO_.5 -> output:#3#3V#0
- U$123, U$162: device SparkFun-MicroMod:MICROMOD_LOGO_.5 -> output:#BYP#0
- U$124: device output:CHG0 -> output:#MEAS#0
- U$125: value (none) -> QWIIC_BOARD_OUTLINESTANDOFF; device output:#3#3V#0 -> SparkFun-Boards:QWIIC_BOARD_MOUNT_SMD_STANDOFFS
- U$126: device output:#BYP#0 -> output:3V30
- U$127: device output:#MEAS#0 -> output:#3#3V_EN#0
- U$128, U$168: value QWIIC_BOARD_OUTLINESTANDOFF -> (none); device SparkFun-Boards:QWIIC_BOARD_MOUNT_SMD_STANDOFFS -> output:#GND#0
- U$129, U$89: device output:3V30 -> output:#GND#0
- U$130, U$170: device output:#3#3V_EN#0 -> output:#CIPO#0
- U$131, U$50, U$91, U$92: device output:#GND#0 -> output:#CIPO#0
- U$132, U$171, U$172, U$211: device output:#GND#0 -> output:#COPI#0
- U$133, U$52, U$93, U$94: device output:#CIPO#0 -> output:#COPI#0
- U$134, U$173, U$174, U$213: device output:#CIPO#0 -> output:#SCK#0
- U$135, U$54, U$95, U$96: device output:#COPI#0 -> output:#SCK#0
- U$136, U$175: device output:#COPI#0 -> output:#VBAT#0
- U$137, U$98: device output:#SCK#0 -> output:#GND#0
- U$138, U$177, U$178, U$217: device output:#SCK#0 -> output:#0
- U$139, U$99: device output:#VBAT#0 -> output:#0
- U$140, U$180: device output:#GND#0 -> buzzard_labels (1):#0
- U$142, U$181, U$182, U$221: device output:#0 -> output:#D0#0
- U$144, U$183, U$184, U$223: device buzzard_labels (1):#0 -> output:#D1#0
- U$146, U$185: device output:#D0#0 -> output:RESET0
- U$148, U$187: device output:#D1#0 -> output:22220
- U$149, U$189: device output:RESET0 -> output:#3#3V#0
- U$151, U$191: device output:22220 -> output:##CS##0
- U$153, U$192, U$193, U$232: device output:#3#3V#0 -> output:##INT##0
- U$155, U$194, U$195, U$234: device output:##CS##0 -> output:QWIIC_CARRIER_#_SINGLE0
- U$157, U$196: device output:##INT##0 -> SparkFun-Aesthetics:SFE_LOGO_FLAME_.2
- U$158, U$198: value QWIIC_BOARD_OUTLINESTANDOFF -> (none); device SparkFun-Boards:QWIIC_BOARD_MOUNT_SMD_STANDOFFS -> SparkFun-MicroMod:MICROMOD_LOGO_.5
- U$160, U$199: device output:QWIIC_CARRIER_#_2X10 -> output:CHG0
- U$161: device SparkFun-Aesthetics:SFE_LOGO_FLAME_.2 -> output:#3#3V#0
- U$163, U$202: device SparkFun-MicroMod:MICROMOD_LOGO_.5 -> output:#MEAS#0
- U$164: value (none) -> QWIIC_BOARD_OUTLINESTANDOFF; device output:CHG0 -> SparkFun-Boards:QWIIC_BOARD_MOUNT_SMD_STANDOFFS
- U$165: device output:#3#3V#0 -> output:3V30
- U$166: device output:#BYP#0 -> output:#3#3V_EN#0
- U$167, U$207: device output:#MEAS#0 -> output:#GND#0
- U$169, U$209: device output:3V30 -> output:#CIPO#0
- U$176, U$215: device output:#COPI#0 -> output:#GND#0
- U$179, U$219: device output:#VBAT#0 -> buzzard_labels (1):#0
- U$186, U$225: device output:#D0#0 -> output:BOOT0
- U$188, U$227, U$228, U$267: device output:#D1#0 -> output:#3#3V#0
- U$19: device output:QWIIC_CARRIER_#_2X10 -> output:QWIIC_CARRIER_#_SINGLE0
- U$190, U$230: device output:BOOT0 -> output:##CS##0
- U$197, U$236, U$237, U$276: device output:##INT##0 -> SparkFun-MicroMod:MICROMOD_LOGO_.5
- U$2, U$78: value QWIIC_BOARD_OUTLINESTANDOFF -> (none); device SparkFun-Boards:QWIIC_BOARD_MOUNT_SMD_STANDOFFS -> output:QWIIC_CARRIER_#_SINGLE0
- U$200, U$239: device output:QWIIC_CARRIER_#_2X10 -> output:#3#3V#0
- U$201: device SparkFun-Aesthetics:SFE_LOGO_FLAME_.2 -> output:#BYP#0
- U$203, U$242: value (none) -> QWIIC_BOARD_OUTLINESTANDOFF; device SparkFun-MicroMod:MICROMOD_LOGO_.5 -> SparkFun-Boards:QWIIC_BOARD_MOUNT_SMD_STANDOFFS
- U$204: device output:CHG0 -> output:3V30
- U$205: device output:#3#3V#0 -> output:#3#3V_EN#0
- U$206, U$246: device output:#BYP#0 -> output:#GND#0
- U$208, U$248: value QWIIC_BOARD_OUTLINESTANDOFF -> (none); device SparkFun-Boards:QWIIC_BOARD_MOUNT_SMD_STANDOFFS -> output:#CIPO#0
- U$210, U$250: device output:#3#3V_EN#0 -> output:#COPI#0
- U$212, U$251, U$252, U$291: device output:#GND#0 -> output:#SCK#0
- U$214, U$253: device output:#CIPO#0 -> output:#VBAT#0
- U$216, U$255, U$256, U$295: device output:#COPI#0 -> output:#0
- U$218, U$257, U$258, U$297: device output:#SCK#0 -> buzzard_labels (1):#0
- U$220, U$260: device output:#GND#0 -> output:#D0#0
- U$222, U$261, U$262, U$301: device output:#0 -> output:#D1#0
- U$224, U$263: device buzzard_labels (1):#0 -> output:RESET0
- U$226, U$265: device output:#D0#0 -> output:22220
- U$229, U$269: device output:RESET0 -> output:##CS##0
- U$231, U$271: device output:22220 -> output:##INT##0
- U$233, U$272, U$273, U$312: device output:#3#3V#0 -> output:QWIIC_CARRIER_#_SINGLE0
- U$235, U$274: device output:##CS##0 -> SparkFun-Aesthetics:SFE_LOGO_FLAME_.2
- U$238: value QWIIC_BOARD_OUTLINESTANDOFF -> (none); device SparkFun-Boards:QWIIC_BOARD_MOUNT_SMD_STANDOFFS -> output:CHG0
- U$240, U$279: device output:QWIIC_CARRIER_#_2X10 -> output:#BYP#0
- U$241: device SparkFun-Aesthetics:SFE_LOGO_FLAME_.2 -> output:#MEAS#0
- U$243, U$282: device SparkFun-MicroMod:MICROMOD_LOGO_.5 -> output:3V30
- U$244: device output:CHG0 -> output:#3#3V_EN#0
- U$245, U$285: device output:#3#3V#0 -> output:#GND#0
- U$247, U$287: device output:#MEAS#0 -> output:#CIPO#0
- U$249, U$289: device output:3V30 -> output:#COPI#0
- U$254, U$293: device output:#CIPO#0 -> output:#GND#0
- U$259, U$299: device output:#VBAT#0 -> output:#D0#0
- U$264, U$303: device buzzard_labels (1):#0 -> output:BOOT0
- U$266, U$305, U$306: device output:#D0#0 -> output:#3#3V#0
- U$268, U$307, U$308: device output:#D1#0 -> output:##CS##0
- U$270, U$310: device output:BOOT0 -> output:##INT##0
- U$275: device output:##CS##0 -> SparkFun-MicroMod:MICROMOD_LOGO_.5
- U$277: device output:##INT##0 -> output:CHG0
- U$278: value QWIIC_BOARD_OUTLINESTANDOFF -> (none); device SparkFun-Boards:QWIIC_BOARD_MOUNT_SMD_STANDOFFS -> output:#3#3V#0
- U$280: device output:QWIIC_CARRIER_#_2X10 -> output:#MEAS#0
- U$281: value (none) -> QWIIC_BOARD_OUTLINESTANDOFF; device SparkFun-Aesthetics:SFE_LOGO_FLAME_.2 -> SparkFun-Boards:QWIIC_BOARD_MOUNT_SMD_STANDOFFS
- U$283: device SparkFun-MicroMod:MICROMOD_LOGO_.5 -> output:#3#3V_EN#0
- U$284: device output:CHG0 -> output:#GND#0
- U$286: device output:#BYP#0 -> output:#CIPO#0
- U$288: value QWIIC_BOARD_OUTLINESTANDOFF -> (none); device SparkFun-Boards:QWIIC_BOARD_MOUNT_SMD_STANDOFFS -> output:#COPI#0
- U$290: device output:#3#3V_EN#0 -> output:#SCK#0
- U$292: device output:#GND#0 -> output:#VBAT#0
- U$294: device output:#CIPO#0 -> output:#0
- U$296: device output:#COPI#0 -> buzzard_labels (1):#0
- U$298: device output:#SCK#0 -> output:#D0#0
- U$300: device output:#GND#0 -> output:#D1#0
- U$302: device output:#0 -> output:RESET0
- U$304: device buzzard_labels (1):#0 -> output:22220
- U$309: device output:RESET0 -> output:##INT##0
- U$311: device output:22220 -> output:QWIIC_CARRIER_#_SINGLE0
- U$40, U$82: device SparkFun-MicroMod:MICROMOD_LOGO_.5 -> output:CHG0
- U$41: device output:CHG0 -> output:#3#3V#0
- U$42: device output:#3#3V#0 -> output:#BYP#0
- U$43: device output:#BYP#0 -> output:#MEAS#0
- U$45: value (none) -> QWIIC_BOARD_OUTLINESTANDOFF; device output:#MEAS#0 -> SparkFun-Boards:QWIIC_BOARD_MOUNT_SMD_STANDOFFS
- U$46: value QWIIC_BOARD_OUTLINESTANDOFF -> (none); device SparkFun-Boards:QWIIC_BOARD_MOUNT_SMD_STANDOFFS -> output:3V30
- U$47: device output:3V30 -> output:#3#3V_EN#0
- U$48, U$90: device output:#3#3V_EN#0 -> output:#GND#0
- U$56, U$97: device output:#SCK#0 -> output:#VBAT#0
- U$57: device output:#VBAT#0 -> output:#GND#0
- U$69: device output:RESET0 -> output:BOOT0
- U$70: device output:BOOT0 -> output:22220
- U$79: device output:QWIIC_CARRIER_#_2X10 -> SparkFun-Aesthetics:SFE_LOGO_FLAME_.2
- U$81: device SparkFun-Aesthetics:SFE_LOGO_FLAME_.2 -> SparkFun-MicroMod:MICROMOD_LOGO_.5
- U$84: device output:CHG0 -> output:#BYP#0
- U$85: device output:#3#3V#0 -> output:#MEAS#0
- U$86: value (none) -> QWIIC_BOARD_OUTLINESTANDOFF; device output:#BYP#0 -> SparkFun-Boards:QWIIC_BOARD_MOUNT_SMD_STANDOFFS
- U$87: device output:#MEAS#0 -> output:3V30
- U$88: value QWIIC_BOARD_OUTLINESTANDOFF -> (none); device SparkFun-Boards:QWIIC_BOARD_MOUNT_SMD_STANDOFFS -> output:#3#3V_EN#0
- moved U$238 203.0 mm to (5.71, 140.0)
- moved U$79 170.3 mm to (18.0, 66.7)
- moved U$239 168.8 mm to (21.0, 141.7), flipped to the bottom
- moved U$160 155.6 mm to (5.71, 103.9), flipped to the top
- moved U$159 153.5 mm to (31.8, 91.6), flipped to the bottom
- moved U$158 149.6 mm to (62.1, 105.5)
- moved U$240 146.8 mm to (11.7, 129.7)
- moved U$235 139.6 mm to (18.0, 138.8), flipped to the top, turned to 0 degrees
- moved U$157 125.2 mm to (18.0, 102.7), flipped to the top, turned to 0 degrees
- moved U$197 114.7 mm to (142.6, 105.5), flipped to the top, turned to 0 degrees
- moved U$237 109.0 mm to (31.8, 127.6), turned to 0 degrees
- moved U$80 104.9 mm to (62.1, 69.5), flipped to the top
- moved U$282 100.8 mm to (86.2, 141.9)
- moved U$275 99.5 mm to (142.6, 141.6), flipped to the top, turned to 0 degrees
- moved U$202 93.6 mm to (97.0, 80.0), flipped to the bottom
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Other:
- board size 239 x 158 mm -> 180.6 x 158 mm
