File: Hardware/Single/Production/MM-Qwiic-Carrier-Single-Panel.brd (EAGLE design)
At the start: 180.6 x 158 mm, 710 parts, among them J12 Vertical Qwiic Connector, J15 MICROMOD-2222-C, J16 MICROMOD-2222-C, J17 QWIIC_RIGHT_ANGLE, J2 QWIIC_RIGHT_ANGLE, J20 Vertical Qwiic Connector, J23 MICROMOD-2222-C, J24 QWIIC_RIGHT_ANGLE, J27 Vertical Qwiic Connector, J30 MICROMOD-2222-C, J31 QWIIC_RIGHT_ANGLE, J34 Vertical Qwiic Connector, J37 MICROMOD-2222-C, J38 QWIIC_RIGHT_ANGLE, J41 Vertical Qwiic Connector, J44 MICROMOD-2222-C, J45 QWIIC_RIGHT_ANGLE, J48 Vertical Qwiic Connector, J5 Vertical Qwiic Connector, J51 MICROMOD-2222-C, J52 QWIIC_RIGHT_ANGLE, J55 Vertical Qwiic Connector, J8 MICROMOD-2222-C, J9 QWIIC_RIGHT_ANGLE, U1 MCP73831, U10 MCP73831, U11 AP7361C-33FGEUDFN-8, U12 MCP73831, U13 AP7361C-33FGEUDFN-8, U14 MCP73831, U15 AP7361C-33FGEUDFN-8, U16 MCP73831, U2 AP7361C-33FGEUDFN-8, U3 MCP73831, U4 AP7361C-33FGEUDFN-8, U5 AP7361C-33FGEUDFN-8, U6 MCP73831, U7 AP7361C-33FGEUDFN-8, U8 MCP73831, U9 AP7361C-33FGEUDFN-8

Commit message: Re-panelized with corrected position silk screen
This is the last time I've got to re-panel hopefully!
Parts:
- moved LOGO14 30.6 mm to (62.2, 82.0)
- moved LOGO20 30.6 mm to (62.2, 118.1)
- moved LOGO3 30.6 mm to (62.2, 9.91)
- moved LOGO8 30.6 mm to (62.2, 46.0)
- moved LOGO11 30.6 mm to (142.7, 46.0)
- moved LOGO17 30.6 mm to (142.7, 82.0)
- moved LOGO23 30.6 mm to (142.7, 118.1)
- moved LOGO5 30.6 mm to (142.7, 9.91)
- moved U$117 30.5 mm to (75.1, 52.1)
- moved U$19 30.5 mm to (75.1, 16.0)
- moved U$195 30.5 mm to (75.1, 88.1)
- moved U$273 30.5 mm to (75.1, 124.2)
- moved LOGO1 30.5 mm to (62.2, 20.8)
- moved LOGO15 30.5 mm to (62.2, 93.0)
- moved LOGO21 30.5 mm to (62.2, 129.0)
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